Commit message: timing script w/rbdl&pybullet ready

File: examples/timing/ur5_rbdl.urdf (robot description, URDF)
Before this commit: robot ur5, 2 links, 1 joints
Links:
- removed link link1
- added link shoulder_link, mass 3.7; collision cylinder length=0.4 radius=0.06; visual cylinder length=0.4 radius=0.06
- added link upper_arm_link, mass 8.393; collision cylinder length=0.4 radius=0.06; visual cylinder length=0.4 radius=0.06
- link base_link: geometry collision cylinder length=0.4 radius=0.06; visual cylinder length=0.4 radius=0.06
Joints:
- added joint shoulder_lift_joint: type revolute, parent shoulder_link, child upper_arm_link, origin xyz=0.0 0.13585 0.0 rpy=0.0 1.57079632679 0.0, axis 1 0 0, limit lower=-6.28318530718 upper=6.28318530718 effort=150.0 velocity=3.15
- joint shoulder_pan_joint: child link1 -> shoulder_link

File: examples/timing/urdf4timing/ur5_rbdl.urdf (robot description, URDF)
Before this commit: robot ur5, 2 links, 1 joints
Links:
- removed link link1
- added link shoulder_link, mass 3.7; collision cylinder length=0.4 radius=0.06; visual cylinder length=0.4 radius=0.06
- link base_link: geometry collision cylinder length=0.4 radius=0.06; visual cylinder length=0.4 radius=0.06
Joints:
- joint shoulder_pan_joint: child link1 -> shoulder_link
