Commit message: timing

File: examples/timing/17dof.urdf (robot description, URDF)
Before this commit: robot ur5, 18 links, 16 joints
Joints:
- added joint wrist_2_joint32: type revolute, parent link16, child link17, origin xyz=0.0 0.093 0.0 rpy=0.0 0.0 0.0, axis 0 0 1, limit lower=-6.28318530718 upper=6.28318530718 effort=28.0 velocity=3.2
- joint wrist_2_joint3: child link17 -> link16; parent link16 -> link15

File: examples/timing/18dof.urdf (robot description, URDF)
Before this commit: robot ur5, 19 links, 17 joints
Joints:
- added joint wrist_2_joint32: type revolute, parent link16, child link17, origin xyz=0.0 0.093 0.0 rpy=0.0 0.0 0.0, axis 0 0 1, limit lower=-6.28318530718 upper=6.28318530718 effort=28.0 velocity=3.2
- joint wrist_2_joint3: child link17 -> link16; parent link16 -> link15

File: examples/timing/20dof.urdf (robot description, URDF)
Before this commit: robot ur5, 21 links, 19 joints
Joints:
- added joint wrist_2_joint32: type revolute, parent link16, child link17, origin xyz=0.0 0.093 0.0 rpy=0.0 0.0 0.0, axis 0 0 1, limit lower=-6.28318530718 upper=6.28318530718 effort=28.0 velocity=3.2
- joint wrist_2_joint3: child link17 -> link16; parent link16 -> link15

File: examples/timing/21dof.urdf (robot description, URDF)
Before this commit: robot ur5, 22 links, 19 joints
Joints:
- added joint shoulder_lift_joint42: type revolute, parent link20, child link21, origin xyz=0.0 0.13585 0.0 rpy=0.0 1.57079632679 0.0, axis 1 0 0, limit lower=-6.28318530718 upper=6.28318530718 effort=150.0 velocity=3.15
- added joint wrist_2_joint32: type revolute, parent link16, child link17, origin xyz=0.0 0.093 0.0 rpy=0.0 0.0 0.0, axis 0 0 1, limit lower=-6.28318530718 upper=6.28318530718 effort=28.0 velocity=3.2
- joint shoulder_lift_joint4: child link21 -> link20; parent link20 -> link19
- joint wrist_2_joint3: child link17 -> link16; parent link16 -> link15

File: examples/timing/22dof.urdf (robot description, URDF)
Before this commit: robot ur5, 23 links, 20 joints
Joints:
- added joint shoulder_lift_joint42: type revolute, parent link20, child link21, origin xyz=0.0 0.13585 0.0 rpy=0.0 1.57079632679 0.0, axis 1 0 0, limit lower=-6.28318530718 upper=6.28318530718 effort=150.0 velocity=3.15
- added joint wrist_2_joint32: type revolute, parent link16, child link17, origin xyz=0.0 0.093 0.0 rpy=0.0 0.0 0.0, axis 0 0 1, limit lower=-6.28318530718 upper=6.28318530718 effort=28.0 velocity=3.2
- joint shoulder_lift_joint4: child link21 -> link20; parent link20 -> link19
- joint wrist_2_joint3: child link17 -> link16; parent link16 -> link15

File: examples/timing/23dof.urdf (robot description, URDF)
Before this commit: robot ur5, 24 links, 21 joints
Joints:
- added joint shoulder_lift_joint42: type revolute, parent link20, child link21, origin xyz=0.0 0.13585 0.0 rpy=0.0 1.57079632679 0.0, axis 1 0 0, limit lower=-6.28318530718 upper=6.28318530718 effort=150.0 velocity=3.15
- added joint wrist_2_joint32: type revolute, parent link16, child link17, origin xyz=0.0 0.093 0.0 rpy=0.0 0.0 0.0, axis 0 0 1, limit lower=-6.28318530718 upper=6.28318530718 effort=28.0 velocity=3.2
- joint shoulder_lift_joint4: child link21 -> link20; parent link20 -> link19
- joint wrist_2_joint3: child link17 -> link16; parent link16 -> link15

File: examples/timing/24dof.urdf (robot description, URDF)
Before this commit: robot ur5, 25 links, 22 joints
Joints:
- added joint shoulder_lift_joint42: type revolute, parent link20, child link21, origin xyz=0.0 0.13585 0.0 rpy=0.0 1.57079632679 0.0, axis 1 0 0, limit lower=-6.28318530718 upper=6.28318530718 effort=150.0 velocity=3.15
- added joint wrist_2_joint32: type revolute, parent link16, child link17, origin xyz=0.0 0.093 0.0 rpy=0.0 0.0 0.0, axis 0 0 1, limit lower=-6.28318530718 upper=6.28318530718 effort=28.0 velocity=3.2
- joint shoulder_lift_joint4: child link21 -> link20; parent link20 -> link19
- joint wrist_2_joint3: child link17 -> link16; parent link16 -> link15

File: examples/timing/25dof.urdf (robot description, URDF)
Before this commit: robot ur5, 20 links, 19 joints
Links:
- added link link20, mass 8.393; collision cylinder length=0.03 radius=0.2; visual cylinder length=0.03 radius=0.2
- added link link21, mass 8.393; collision cylinder length=0.03 radius=0.2; visual cylinder length=0.03 radius=0.2
- added link link22, mass 2.275; collision cylinder length=0.03 radius=0.2; visual cylinder length=0.03 radius=0.2
- added link link23, mass 1.219; collision cylinder length=0.03 radius=0.2; visual cylinder length=0.03 radius=0.2
- added link link24, mass 1.219; collision cylinder length=0.03 radius=0.2; visual cylinder length=0.03 radius=0.2
- added link link25, mass 0.1879; collision cylinder length=0.03 radius=0.2; visual cylinder length=0.03 radius=0.2
Joints:
- added joint elbow_joint4: type revolute, parent link21, child link22, origin xyz=0.0 -0.1197 0.425 rpy=0.0 0.0 0.0, axis 0 -1.0 0, limit lower=-3.14159265359 upper=3.14159265359 effort=150.0 velocity=3.15
- added joint shoulder_lift_joint4: type revolute, parent link19, child link20, origin xyz=0.0 0.13585 0.0 rpy=0.0 1.57079632679 0.0, axis 1 0 0, limit lower=-6.28318530718 upper=6.28318530718 effort=150.0 velocity=3.15
- added joint shoulder_lift_joint42: type revolute, parent link20, child link21, origin xyz=0.0 0.13585 0.0 rpy=0.0 1.57079632679 0.0, axis 1 0 0, limit lower=-6.28318530718 upper=6.28318530718 effort=150.0 velocity=3.15
- added joint wrist_1_joint4: type revolute, parent link22, child link23, origin xyz=0.0 0.0 0.39225 rpy=0.0 1.57079632679 0.0, axis 0 1 0, limit lower=-6.28318530718 upper=6.28318530718 effort=28.0 velocity=3.2
- added joint wrist_2_joint4: type revolute, parent link23, child link24, origin xyz=0.0 0.093 0.0 rpy=0.0 0.0 0.0, axis 0 0 1, limit lower=-6.28318530718 upper=6.28318530718 effort=28.0 velocity=3.2
- added joint wrist_3_joint4: type revolute, parent link24, child link25, origin xyz=0.0 0.0 0.09465 rpy=0.0 0.0 0.0, axis 0 1 0, limit lower=-6.28318530718 upper=6.28318530718 effort=28.0 velocity=3.2

File: examples/timing/26dof.urdf (robot description, URDF)
Before this commit: robot ur5, 20 links, 19 joints
Links:
- added link link20, mass 8.393; collision cylinder length=0.03 radius=0.2; visual cylinder length=0.03 radius=0.2
- added link link21, mass 8.393; collision cylinder length=0.03 radius=0.2; visual cylinder length=0.03 radius=0.2
- added link link22, mass 2.275; collision cylinder length=0.03 radius=0.2; visual cylinder length=0.03 radius=0.2
- added link link23, mass 1.219; collision cylinder length=0.03 radius=0.2; visual cylinder length=0.03 radius=0.2
- added link link24, mass 1.219; collision cylinder length=0.03 radius=0.2; visual cylinder length=0.03 radius=0.2
- added link link25, mass 0.1879; collision cylinder length=0.03 radius=0.2; visual cylinder length=0.03 radius=0.2
- added link link26, mass 3.7; collision cylinder length=0.03 radius=0.2; visual cylinder length=0.03 radius=0.2
Joints:
- added joint elbow_joint4: type revolute, parent link21, child link22, origin xyz=0.0 -0.1197 0.425 rpy=0.0 0.0 0.0, axis 0 -1.0 0, limit lower=-3.14159265359 upper=3.14159265359 effort=150.0 velocity=3.15
- added joint shoulder_lift_joint4: type revolute, parent link19, child link20, origin xyz=0.0 0.13585 0.0 rpy=0.0 1.57079632679 0.0, axis 1 0 0, limit lower=-6.28318530718 upper=6.28318530718 effort=150.0 velocity=3.15
- added joint shoulder_lift_joint42: type revolute, parent link20, child link21, origin xyz=0.0 0.13585 0.0 rpy=0.0 1.57079632679 0.0, axis 1 0 0, limit lower=-6.28318530718 upper=6.28318530718 effort=150.0 velocity=3.15
- added joint shoulder_pan_joint5: type revolute, parent link25, child link26, origin xyz=0.0 0.0 0.089159 rpy=0.0 0.0 0.0, axis 0 0 1, limit lower=-6.28318530718 upper=6.28318530718 effort=150.0 velocity=3.15
- added joint wrist_1_joint4: type revolute, parent link22, child link23, origin xyz=0.0 0.0 0.39225 rpy=0.0 1.57079632679 0.0, axis 0 1 0, limit lower=-6.28318530718 upper=6.28318530718 effort=28.0 velocity=3.2
- added joint wrist_2_joint4: type revolute, parent link23, child link24, origin xyz=0.0 0.093 0.0 rpy=0.0 0.0 0.0, axis 0 0 1, limit lower=-6.28318530718 upper=6.28318530718 effort=28.0 velocity=3.2
- added joint wrist_3_joint4: type revolute, parent link24, child link25, origin xyz=0.0 0.0 0.09465 rpy=0.0 0.0 0.0, axis 0 1 0, limit lower=-6.28318530718 upper=6.28318530718 effort=28.0 velocity=3.2

File: examples/timing/27dof.urdf (robot description, URDF)
Before this commit: robot ur5, 20 links, 19 joints
Links:
- added link link20, mass 8.393; collision cylinder length=0.03 radius=0.2; visual cylinder length=0.03 radius=0.2
- added link link21, mass 8.393; collision cylinder length=0.03 radius=0.2; visual cylinder length=0.03 radius=0.2
- added link link22, mass 2.275; collision cylinder length=0.03 radius=0.2; visual cylinder length=0.03 radius=0.2
- added link link23, mass 1.219; collision cylinder length=0.03 radius=0.2; visual cylinder length=0.03 radius=0.2
- added link link24, mass 1.219; collision cylinder length=0.03 radius=0.2; visual cylinder length=0.03 radius=0.2
- added link link25, mass 0.1879; collision cylinder length=0.03 radius=0.2; visual cylinder length=0.03 radius=0.2
- added link link26, mass 3.7; collision cylinder length=0.03 radius=0.2; visual cylinder length=0.03 radius=0.2
- added link link27, mass 8.393; collision cylinder length=0.03 radius=0.2; visual cylinder length=0.03 radius=0.2
Joints:
- added joint elbow_joint4: type revolute, parent link21, child link22, origin xyz=0.0 -0.1197 0.425 rpy=0.0 0.0 0.0, axis 0 -1.0 0, limit lower=-3.14159265359 upper=3.14159265359 effort=150.0 velocity=3.15
- added joint shoulder_lift_joint4: type revolute, parent link19, child link20, origin xyz=0.0 0.13585 0.0 rpy=0.0 1.57079632679 0.0, axis 1 0 0, limit lower=-6.28318530718 upper=6.28318530718 effort=150.0 velocity=3.15
- added joint shoulder_lift_joint42: type revolute, parent link20, child link21, origin xyz=0.0 0.13585 0.0 rpy=0.0 1.57079632679 0.0, axis 1 0 0, limit lower=-6.28318530718 upper=6.28318530718 effort=150.0 velocity=3.15
- added joint shoulder_lift_joint5: type revolute, parent link26, child link27, origin xyz=0.0 0.13585 0.0 rpy=0.0 1.57079632679 0.0, axis 1 0 0, limit lower=-6.28318530718 upper=6.28318530718 effort=150.0 velocity=3.15
- added joint shoulder_pan_joint5: type revolute, parent link25, child link26, origin xyz=0.0 0.0 0.089159 rpy=0.0 0.0 0.0, axis 0 0 1, limit lower=-6.28318530718 upper=6.28318530718 effort=150.0 velocity=3.15
- added joint wrist_1_joint4: type revolute, parent link22, child link23, origin xyz=0.0 0.0 0.39225 rpy=0.0 1.57079632679 0.0, axis 0 1 0, limit lower=-6.28318530718 upper=6.28318530718 effort=28.0 velocity=3.2
- added joint wrist_2_joint4: type revolute, parent link23, child link24, origin xyz=0.0 0.093 0.0 rpy=0.0 0.0 0.0, axis 0 0 1, limit lower=-6.28318530718 upper=6.28318530718 effort=28.0 velocity=3.2
- added joint wrist_3_joint4: type revolute, parent link24, child link25, origin xyz=0.0 0.0 0.09465 rpy=0.0 0.0 0.0, axis 0 1 0, limit lower=-6.28318530718 upper=6.28318530718 effort=28.0 velocity=3.2

File: examples/timing/28dof.urdf (robot description, URDF)
Before this commit: robot ur5, 20 links, 19 joints
Links:
- added link link20, mass 8.393; collision cylinder length=0.03 radius=0.2; visual cylinder length=0.03 radius=0.2
- added link link21, mass 8.393; collision cylinder length=0.03 radius=0.2; visual cylinder length=0.03 radius=0.2
- added link link22, mass 2.275; collision cylinder length=0.03 radius=0.2; visual cylinder length=0.03 radius=0.2
- added link link23, mass 1.219; collision cylinder length=0.03 radius=0.2; visual cylinder length=0.03 radius=0.2
- added link link24, mass 1.219; collision cylinder length=0.03 radius=0.2; visual cylinder length=0.03 radius=0.2
- added link link25, mass 0.1879; collision cylinder length=0.03 radius=0.2; visual cylinder length=0.03 radius=0.2
- added link link26, mass 3.7; collision cylinder length=0.03 radius=0.2; visual cylinder length=0.03 radius=0.2
- added link link27, mass 8.393; collision cylinder length=0.03 radius=0.2; visual cylinder length=0.03 radius=0.2
- added link link28, mass 2.275; collision cylinder length=0.03 radius=0.2; visual cylinder length=0.03 radius=0.2
Joints:
- added joint elbow_joint4: type revolute, parent link21, child link22, origin xyz=0.0 -0.1197 0.425 rpy=0.0 0.0 0.0, axis 0 -1.0 0, limit lower=-3.14159265359 upper=3.14159265359 effort=150.0 velocity=3.15
- added joint elbow_joint5: type revolute, parent link27, child link28, origin xyz=0.0 -0.1197 0.425 rpy=0.0 0.0 0.0, axis 0 -1.0 0, limit lower=-3.14159265359 upper=3.14159265359 effort=150.0 velocity=3.15
- added joint shoulder_lift_joint4: type revolute, parent link19, child link20, origin xyz=0.0 0.13585 0.0 rpy=0.0 1.57079632679 0.0, axis 1 0 0, limit lower=-6.28318530718 upper=6.28318530718 effort=150.0 velocity=3.15
- added joint shoulder_lift_joint42: type revolute, parent link20, child link21, origin xyz=0.0 0.13585 0.0 rpy=0.0 1.57079632679 0.0, axis 1 0 0, limit lower=-6.28318530718 upper=6.28318530718 effort=150.0 velocity=3.15
- added joint shoulder_lift_joint5: type revolute, parent link26, child link27, origin xyz=0.0 0.13585 0.0 rpy=0.0 1.57079632679 0.0, axis 1 0 0, limit lower=-6.28318530718 upper=6.28318530718 effort=150.0 velocity=3.15
- added joint shoulder_pan_joint5: type revolute, parent link25, child link26, origin xyz=0.0 0.0 0.089159 rpy=0.0 0.0 0.0, axis 0 0 1, limit lower=-6.28318530718 upper=6.28318530718 effort=150.0 velocity=3.15
- added joint wrist_1_joint4: type revolute, parent link22, child link23, origin xyz=0.0 0.0 0.39225 rpy=0.0 1.57079632679 0.0, axis 0 1 0, limit lower=-6.28318530718 upper=6.28318530718 effort=28.0 velocity=3.2
- added joint wrist_2_joint4: type revolute, parent link23, child link24, origin xyz=0.0 0.093 0.0 rpy=0.0 0.0 0.0, axis 0 0 1, limit lower=-6.28318530718 upper=6.28318530718 effort=28.0 velocity=3.2
- added joint wrist_3_joint4: type revolute, parent link24, child link25, origin xyz=0.0 0.0 0.09465 rpy=0.0 0.0 0.0, axis 0 1 0, limit lower=-6.28318530718 upper=6.28318530718 effort=28.0 velocity=3.2

File: examples/timing/29dof.urdf (robot description, URDF)
Before this commit: robot ur5, 20 links, 19 joints
Links:
- added link link20, mass 8.393; collision cylinder length=0.03 radius=0.2; visual cylinder length=0.03 radius=0.2
- added link link21, mass 8.393; collision cylinder length=0.03 radius=0.2; visual cylinder length=0.03 radius=0.2
- added link link22, mass 2.275; collision cylinder length=0.03 radius=0.2; visual cylinder length=0.03 radius=0.2
- added link link23, mass 1.219; collision cylinder length=0.03 radius=0.2; visual cylinder length=0.03 radius=0.2
- added link link24, mass 1.219; collision cylinder length=0.03 radius=0.2; visual cylinder length=0.03 radius=0.2
- added link link25, mass 0.1879; collision cylinder length=0.03 radius=0.2; visual cylinder length=0.03 radius=0.2
- added link link26, mass 3.7; collision cylinder length=0.03 radius=0.2; visual cylinder length=0.03 radius=0.2
- added link link27, mass 8.393; collision cylinder length=0.03 radius=0.2; visual cylinder length=0.03 radius=0.2
- added link link28, mass 2.275; collision cylinder length=0.03 radius=0.2; visual cylinder length=0.03 radius=0.2
- added link link29, mass 1.219; collision cylinder length=0.03 radius=0.2; visual cylinder length=0.03 radius=0.2
Joints:
- added joint elbow_joint4: type revolute, parent link21, child link22, origin xyz=0.0 -0.1197 0.425 rpy=0.0 0.0 0.0, axis 0 -1.0 0, limit lower=-3.14159265359 upper=3.14159265359 effort=150.0 velocity=3.15
- added joint elbow_joint5: type revolute, parent link27, child link28, origin xyz=0.0 -0.1197 0.425 rpy=0.0 0.0 0.0, axis 0 -1.0 0, limit lower=-3.14159265359 upper=3.14159265359 effort=150.0 velocity=3.15
- added joint shoulder_lift_joint4: type revolute, parent link19, child link20, origin xyz=0.0 0.13585 0.0 rpy=0.0 1.57079632679 0.0, axis 1 0 0, limit lower=-6.28318530718 upper=6.28318530718 effort=150.0 velocity=3.15
- added joint shoulder_lift_joint42: type revolute, parent link20, child link21, origin xyz=0.0 0.13585 0.0 rpy=0.0 1.57079632679 0.0, axis 1 0 0, limit lower=-6.28318530718 upper=6.28318530718 effort=150.0 velocity=3.15
- added joint shoulder_lift_joint5: type revolute, parent link26, child link27, origin xyz=0.0 0.13585 0.0 rpy=0.0 1.57079632679 0.0, axis 1 0 0, limit lower=-6.28318530718 upper=6.28318530718 effort=150.0 velocity=3.15
- added joint shoulder_pan_joint5: type revolute, parent link25, child link26, origin xyz=0.0 0.0 0.089159 rpy=0.0 0.0 0.0, axis 0 0 1, limit lower=-6.28318530718 upper=6.28318530718 effort=150.0 velocity=3.15
- added joint wrist_1_joint4: type revolute, parent link22, child link23, origin xyz=0.0 0.0 0.39225 rpy=0.0 1.57079632679 0.0, axis 0 1 0, limit lower=-6.28318530718 upper=6.28318530718 effort=28.0 velocity=3.2
- added joint wrist_1_joint5: type revolute, parent link28, child link29, origin xyz=0.0 0.0 0.39225 rpy=0.0 1.57079632679 0.0, axis 0 1 0, limit lower=-6.28318530718 upper=6.28318530718 effort=28.0 velocity=3.2
- added joint wrist_2_joint4: type revolute, parent link23, child link24, origin xyz=0.0 0.093 0.0 rpy=0.0 0.0 0.0, axis 0 0 1, limit lower=-6.28318530718 upper=6.28318530718 effort=28.0 velocity=3.2
- added joint wrist_3_joint4: type revolute, parent link24, child link25, origin xyz=0.0 0.0 0.09465 rpy=0.0 0.0 0.0, axis 0 1 0, limit lower=-6.28318530718 upper=6.28318530718 effort=28.0 velocity=3.2

File: examples/timing/30dof.urdf (robot description, URDF)
Before this commit: robot ur5, 20 links, 19 joints
Links:
- added link link20, mass 8.393; collision cylinder length=0.03 radius=0.2; visual cylinder length=0.03 radius=0.2
- added link link21, mass 8.393; collision cylinder length=0.03 radius=0.2; visual cylinder length=0.03 radius=0.2
- added link link22, mass 2.275; collision cylinder length=0.03 radius=0.2; visual cylinder length=0.03 radius=0.2
- added link link23, mass 1.219; collision cylinder length=0.03 radius=0.2; visual cylinder length=0.03 radius=0.2
- added link link24, mass 1.219; collision cylinder length=0.03 radius=0.2; visual cylinder length=0.03 radius=0.2
- added link link25, mass 0.1879; collision cylinder length=0.03 radius=0.2; visual cylinder length=0.03 radius=0.2
- added link link26, mass 3.7; collision cylinder length=0.03 radius=0.2; visual cylinder length=0.03 radius=0.2
- added link link27, mass 8.393; collision cylinder length=0.03 radius=0.2; visual cylinder length=0.03 radius=0.2
- added link link28, mass 2.275; collision cylinder length=0.03 radius=0.2; visual cylinder length=0.03 radius=0.2
- added link link29, mass 1.219; collision cylinder length=0.03 radius=0.2; visual cylinder length=0.03 radius=0.2
- added link link30, mass 1.219; collision cylinder length=0.03 radius=0.2; visual cylinder length=0.03 radius=0.2
Joints:
- added joint elbow_joint4: type revolute, parent link21, child link22, origin xyz=0.0 -0.1197 0.425 rpy=0.0 0.0 0.0, axis 0 -1.0 0, limit lower=-3.14159265359 upper=3.14159265359 effort=150.0 velocity=3.15
- added joint elbow_joint5: type revolute, parent link27, child link28, origin xyz=0.0 -0.1197 0.425 rpy=0.0 0.0 0.0, axis 0 -1.0 0, limit lower=-3.14159265359 upper=3.14159265359 effort=150.0 velocity=3.15
- added joint shoulder_lift_joint4: type revolute, parent link19, child link20, origin xyz=0.0 0.13585 0.0 rpy=0.0 1.57079632679 0.0, axis 1 0 0, limit lower=-6.28318530718 upper=6.28318530718 effort=150.0 velocity=3.15
- added joint shoulder_lift_joint42: type revolute, parent link20, child link21, origin xyz=0.0 0.13585 0.0 rpy=0.0 1.57079632679 0.0, axis 1 0 0, limit lower=-6.28318530718 upper=6.28318530718 effort=150.0 velocity=3.15
- added joint shoulder_lift_joint5: type revolute, parent link26, child link27, origin xyz=0.0 0.13585 0.0 rpy=0.0 1.57079632679 0.0, axis 1 0 0, limit lower=-6.28318530718 upper=6.28318530718 effort=150.0 velocity=3.15
- added joint shoulder_pan_joint5: type revolute, parent link25, child link26, origin xyz=0.0 0.0 0.089159 rpy=0.0 0.0 0.0, axis 0 0 1, limit lower=-6.28318530718 upper=6.28318530718 effort=150.0 velocity=3.15
- added joint wrist_1_joint4: type revolute, parent link22, child link23, origin xyz=0.0 0.0 0.39225 rpy=0.0 1.57079632679 0.0, axis 0 1 0, limit lower=-6.28318530718 upper=6.28318530718 effort=28.0 velocity=3.2
- added joint wrist_1_joint5: type revolute, parent link28, child link29, origin xyz=0.0 0.0 0.39225 rpy=0.0 1.57079632679 0.0, axis 0 1 0, limit lower=-6.28318530718 upper=6.28318530718 effort=28.0 velocity=3.2
- added joint wrist_2_joint4: type revolute, parent link23, child link24, origin xyz=0.0 0.093 0.0 rpy=0.0 0.0 0.0, axis 0 0 1, limit lower=-6.28318530718 upper=6.28318530718 effort=28.0 velocity=3.2
- added joint wrist_2_joint5: type revolute, parent link29, child link30, origin xyz=0.0 0.093 0.0 rpy=0.0 0.0 0.0, axis 0 0 1, limit lower=-6.28318530718 upper=6.28318530718 effort=28.0 velocity=3.2
- added joint wrist_3_joint4: type revolute, parent link24, child link25, origin xyz=0.0 0.0 0.09465 rpy=0.0 0.0 0.0, axis 0 1 0, limit lower=-6.28318530718 upper=6.28318530718 effort=28.0 velocity=3.2
