Commit message: timing

File: examples/timing/26dof.urdf (robot description, URDF)
Before this commit: robot ur5, 27 links, 26 joints
Links:
- link link26: mass 3.7 -> 0.1879
Joints:
- removed joint shoulder_pan_joint5
- added joint wrist_3_joint42: type revolute, parent link25, child link26, origin xyz=0.0 0.0 0.09465 rpy=0.0 0.0 0.0, axis 0 1 0, limit lower=-6.28318530718 upper=6.28318530718 effort=28.0 velocity=3.2
