Commit message: added gravity

File: examples/urdf/ur5.urdf (robot description, URDF)
Before this commit: robot ur5, 11 links, 10 joints
Links:
- link forearm_link: mass 2.275 -> None
- link shoulder_link: mass 3.7 -> None
- link upper_arm_link: mass 8.393 -> None
Joints:
- joint elbow_joint: axis 0 1 0 -> 0 -1.0 0

Commit message: added some fixed joint functionality

File: examples/urdf/ur5.urdf (robot description, URDF)
Before this commit: robot ur5, 11 links, 10 joints
Joints:
- joint shoulder_lift_joint: axis 0 1 0 -> 0 0 0; type revolute -> fixed

Commit message: Added ur5 examples

File: examples/urdf/ur5.urdf (robot description, URDF)
Before this commit: robot ur5, 11 links, 10 joints
Joints:
- joint shoulder_lift_joint: type fixed -> revolute

Commit message: changed names and added numerical tests

File: examples/urdf/ur5.urdf (robot description, URDF)
Before this commit: robot ur5, 11 links, 10 joints
Links:
- link forearm_link: mass None -> 2.275
- link shoulder_link: mass None -> 3.7
Joints:
- joint shoulder_lift_joint: axis 0 0 0 -> 0 0 1
