Commit message: timing & numerical

File: examples/urdf/gantry.urdf (robot description, URDF)
Before this commit: robot gantry, 14 links, 13 joints
Links:
- removed link gantry_root
- link gantry_base_link: geometry collision cylinder length=0.104 radius=0.06; visual cylinder length=0.104 radius=0.06
- link gantry_link_1: geometry collision cylinder length=0.104 radius=0.06; visual cylinder length=0.104 radius=0.06
- link gantry_link_2: geometry collision cylinder length=0.104 radius=0.06; visual cylinder length=0.104 radius=0.06
- link gantry_link_3: geometry collision cylinder length=0.104 radius=0.06; visual cylinder length=0.104 radius=0.06
- link gantry_link_4: geometry collision cylinder length=0.104 radius=0.06; visual cylinder length=0.104 radius=0.06
- link gantry_link_5: geometry collision cylinder length=0.104 radius=0.06; visual cylinder length=0.104 radius=0.06
- link gantry_link_6: geometry collision cylinder length=0.104 radius=0.06; visual cylinder length=0.104 radius=0.06
- link gantry_link_arm: geometry collision cylinder length=0.104 radius=0.06; visual cylinder length=0.104 radius=0.06
- link gantry_link_base: geometry collision cylinder length=0.104 radius=0.06; visual cylinder length=0.104 radius=0.06
- link gantry_link_leg: geometry collision cylinder length=0.104 radius=0.06; visual cylinder length=0.104 radius=0.06
- link gantry_link_trolley: geometry collision cylinder length=0.104 radius=0.06; visual cylinder length=0.104 radius=0.06
- link gantry_robot_connection: mass None -> 2
Joints:
- removed joint gantry_joint_base

File: examples/urdf/kuka_modified.urdf (robot description, URDF)
Before this commit: robot kuka_lwr, 8 links, 7 joints
Links:
- link calib_kuka_arm_base_link: geometry 
- link kuka_arm_1_link: geometry 
- link kuka_arm_2_link: geometry 
- link kuka_arm_3_link: geometry 
- link kuka_arm_4_link: geometry 
- link kuka_arm_5_link: geometry 
- link kuka_arm_6_link: geometry 
- link kuka_arm_7_link: geometry 

File: examples/urdf/kukalwr.urdf (robot description, URDF)
Before this commit: robot kuka_lwr, 8 links, 7 joints
Links:
- link calib_kuka_arm_base_link: geometry 
- link kuka_arm_1_link: geometry 
- link kuka_arm_2_link: geometry 
- link kuka_arm_3_link: geometry 
- link kuka_arm_4_link: geometry 
- link kuka_arm_5_link: geometry 
- link kuka_arm_6_link: geometry 
- link kuka_arm_7_link: geometry 

File: examples/urdf/pantilt.urdf (robot description, URDF)
Before this commit: robot pan_tilt, 3 links, 2 joints
Links:
- link base_link: geometry 
- link pan_link: geometry 
- link tilt_link: geometry 
Joints:
- joint pan_joint: origin xyz=0.0 0.0 0 rpy=0.0 0.0 0.0 -> xyz=0.0 0.0 1.0 rpy=0.0 0.0 0.0
