Commit message: minor changes & fixed docstrings.

File: examples/urdf/pantilt.urdf (robot description, URDF)
Before this commit: robot pan_tilt, 3 links, 2 joints
Links:
- link base_link: geometry collision cylinder length=0.03 radius=0.2; visual cylinder length=0.01 radius=0.2
- link pan_link: geometry collision cylinder length=0.4 radius=0.06; visual cylinder length=0.4 radius=0.04
- link tilt_link: mass 5 -> 1; geometry collision cylinder length=0.4 radius=0.06; visual cylinder length=0.4 radius=0.04
Joints:
- joint tilt_joint: axis 0.0 1.0 0.0 -> 0 1 0; limit lower=-4.64 upper=4.64 effort=300 velocity=1.0 -> lower=-4.64 upper=-1.5 effort=300 velocity=0.1; origin xyz=4 0 1 rpy=0.0 0.0 0.0 -> xyz=0 0 0.2

File: examples/urdf/snake_robot.urdf (robot description, URDF)
Before this commit: robot snake_robot, 17 links, 16 joints
Links:
- link base_link: geometry collision cylinder length=0.62 radius=0.35297; visual cylinder length=0.62 radius=0.35297
