Commit message: usr ex

File: examples/timing/urdf4timing/34dof.urdf (robot description, URDF)
Before this commit: robot ur5, 35 links, 32 joints
Links:
- removed link forearm_link
- removed link shoulder_link
- removed link shoulder_link3
- removed link upper_arm_link
- removed link upper_arm_link2
- removed link wrist_1_link
- removed link wrist_2_link
- added link link1, mass 3.7; collision cylinder length=0.03 radius=0.2; visual cylinder length=0.03 radius=0.2
- added link link12, mass 3.7; collision cylinder length=0.03 radius=0.2; visual cylinder length=0.03 radius=0.2
- added link link2, mass 8.393; collision cylinder length=0.03 radius=0.2; visual cylinder length=0.03 radius=0.2
- added link link3, mass 2.275; collision cylinder length=0.03 radius=0.2; visual cylinder length=0.03 radius=0.2
- added link link4, mass 1.219; collision cylinder length=0.03 radius=0.2; visual cylinder length=0.03 radius=0.2
- added link link5, mass 1.219; collision cylinder length=0.03 radius=0.2; visual cylinder length=0.03 radius=0.2
- added link link7, mass 8.393; collision cylinder length=0.03 radius=0.2; visual cylinder length=0.03 radius=0.2
- link base_link: geometry collision cylinder length=0.03 radius=0.2; visual cylinder length=0.03 radius=0.2
- link link10: geometry collision cylinder length=0.03 radius=0.2; visual cylinder length=0.03 radius=0.2
- link link11: geometry collision cylinder length=0.03 radius=0.2; visual cylinder length=0.03 radius=0.2
- link link13: geometry collision cylinder length=0.03 radius=0.2; visual cylinder length=0.03 radius=0.2
- link link14: geometry collision cylinder length=0.03 radius=0.2; visual cylinder length=0.03 radius=0.2
- link link15: geometry collision cylinder length=0.03 radius=0.2; visual cylinder length=0.03 radius=0.2
- link link16: geometry collision cylinder length=0.03 radius=0.2; visual cylinder length=0.03 radius=0.2
- link link17: geometry collision cylinder length=0.03 radius=0.2; visual cylinder length=0.03 radius=0.2
- link link18: geometry collision cylinder length=0.03 radius=0.2; visual cylinder length=0.03 radius=0.2
- link link19: geometry collision cylinder length=0.03 radius=0.2; visual cylinder length=0.03 radius=0.2
- link link20: mass 8.393 -> 4.393; geometry collision cylinder length=0.03 radius=0.2; visual cylinder length=0.03 radius=0.2
- link link21: geometry collision cylinder length=0.03 radius=0.2; visual cylinder length=0.03 radius=0.2
- link link22: geometry collision cylinder length=0.03 radius=0.2; visual cylinder length=0.03 radius=0.2
- link link23: geometry collision cylinder length=0.03 radius=0.2; visual cylinder length=0.03 radius=0.2
- link link24: geometry collision cylinder length=0.03 radius=0.2; visual cylinder length=0.03 radius=0.2
- link link25: geometry collision cylinder length=0.03 radius=0.2; visual cylinder length=0.03 radius=0.2
- link link26: geometry collision cylinder length=0.03 radius=0.2; visual cylinder length=0.03 radius=0.2
- link link27: mass None -> 8.393; geometry collision cylinder length=0.03 radius=0.2; visual cylinder length=0.03 radius=0.2
- link link28: geometry collision cylinder length=0.03 radius=0.2; visual cylinder length=0.03 radius=0.2
- link link29: geometry collision cylinder length=0.03 radius=0.2; visual cylinder length=0.03 radius=0.2
- link link30: geometry collision cylinder length=0.03 radius=0.2; visual cylinder length=0.03 radius=0.2
- link link31: geometry collision cylinder length=0.03 radius=0.2; visual cylinder length=0.03 radius=0.2
- link link32: geometry collision cylinder length=0.03 radius=0.2; visual cylinder length=0.03 radius=0.2
- link link33: mass 8.393 -> 3.7; geometry collision cylinder length=0.03 radius=0.2; visual cylinder length=0.03 radius=0.2
- link link34: mass 2.275 -> 8.393; geometry collision cylinder length=0.03 radius=0.2; visual cylinder length=0.03 radius=0.2
- link link6: geometry collision cylinder length=0.03 radius=0.2; visual cylinder length=0.03 radius=0.2
- link link8: geometry collision cylinder length=0.03 radius=0.2; visual cylinder length=0.03 radius=0.2
- link link9: geometry collision cylinder length=0.03 radius=0.2; visual cylinder length=0.03 radius=0.2
Joints:
- removed joint elbow_joint
- removed joint elbow_joint2
- removed joint elbow_joint3
- removed joint elbow_joint4
- removed joint elbow_joint5
- removed joint elbow_joint6
- removed joint shoulder_lift_joint
- removed joint shoulder_lift_joint2
- removed joint shoulder_lift_joint3
- removed joint shoulder_lift_joint4
- removed joint shoulder_lift_joint5
- removed joint shoulder_lift_joint6
- removed joint shoulder_pan_joint
- removed joint shoulder_pan_joint3
- removed joint shoulder_pan_joint4
- removed joint shoulder_pan_joint5
- removed joint shoulder_pan_joint6
- removed joint wrist_1_joint
- removed joint wrist_1_joint2
- removed joint wrist_1_joint3
- removed joint wrist_1_joint4
- removed joint wrist_1_joint5
- removed joint wrist_2_joint
- removed joint wrist_2_joint2
- removed joint wrist_2_joint3
- removed joint wrist_2_joint4
- removed joint wrist_2_joint5
- removed joint wrist_3_joint
- removed joint wrist_3_joint2
- removed joint wrist_3_joint3
- removed joint wrist_3_joint4
- removed joint wrist_3_joint5
- added joint joint1: type revolute, parent base_link, child link1, origin xyz=0.0 0.0 0.089159 rpy=0.0 0.0 0.0, axis 1 0 0, limit lower=-6.28318530718 upper=6.28318530718 effort=150.0 velocity=3.15
- added joint joint10: type revolute, parent link9, child link10, origin xyz=0.0 0.093 0.0 rpy=0.0 0.0 0.0, axis 0 0 1, limit lower=-6.28318530718 upper=6.28318530718 effort=28.0 velocity=3.2
- added joint joint11: type revolute, parent link10, child link11, origin xyz=0.0 0.0 0.09465 rpy=0.0 0.0 0.0, axis 0 1 0, limit lower=-6.28318530718 upper=6.28318530718 effort=28.0 velocity=3.2
- added joint joint12: type revolute, parent link11, child link12, origin xyz=0.0 0.0 0.089159 rpy=0.0 0.0 0.0, axis 0 0 1, limit lower=-6.28318530718 upper=6.28318530718 effort=150.0 velocity=3.15
- added joint joint13: type revolute, parent link12, child link13, origin xyz=0.0 0.13585 0.0 rpy=0.0 1.57079632679 0.0, axis 1 0 0, limit lower=-6.28318530718 upper=6.28318530718 effort=150.0 velocity=3.15
- added joint joint14: type revolute, parent link13, child link14, origin xyz=0.0 -0.1197 0.425 rpy=0.0 0.0 0.0, axis 0 -1.0 0, limit lower=-3.14159265359 upper=3.14159265359 effort=150.0 velocity=3.15
- added joint joint15: type revolute, parent link14, child link15, origin xyz=0.0 0.0 0.39225 rpy=0.0 1.57079632679 0.0, axis 0 1 0, limit lower=-6.28318530718 upper=6.28318530718 effort=28.0 velocity=3.2
- added joint joint16: type revolute, parent link15, child link16, origin xyz=0.0 0.093 0.0 rpy=0.0 0.0 0.0, axis 0 0 1, limit lower=-6.28318530718 upper=6.28318530718 effort=28.0 velocity=3.2
- added joint joint17: type revolute, parent link16, child link17, origin xyz=0.0 0.093 0.0 rpy=0.0 0.0 0.0, axis 0 0 1, limit lower=-6.28318530718 upper=6.28318530718 effort=28.0 velocity=3.2
- added joint joint18: type revolute, parent link17, child link18, origin xyz=0.0 0.0 0.09465 rpy=0.0 0.0 0.0, axis 0 1 0, limit lower=-6.28318530718 upper=6.28318530718 effort=28.0 velocity=3.2
- added joint joint19: type revolute, parent link18, child link19, origin xyz=0.0 0.0 0.089159 rpy=0.0 0.0 0.0, axis 0 0 1, limit lower=-6.28318530718 upper=6.28318530718 effort=150.0 velocity=3.15
- added joint joint2: type revolute, parent link1, child link2, origin xyz=0.0 0.13585 0.0 rpy=0.0 1.57079632679 0.0, axis 1 0 0, limit lower=-6.28318530718 upper=6.28318530718 effort=150.0 velocity=3.15
- added joint joint20: type revolute, parent link19, child link20, origin xyz=0.0 0.13585 0.0 rpy=0.0 1.57079632679 0.0, axis 1 0 0, limit lower=-6.28318530718 upper=6.28318530718 effort=150.0 velocity=3.15
- added joint joint21: type revolute, parent link20, child link21, origin xyz=0.0 0.13585 0.0 rpy=0.0 1.57079632679 0.0, axis 1 0 0, limit lower=-6.28318530718 upper=6.28318530718 effort=150.0 velocity=3.15
- added joint joint22: type revolute, parent link21, child link22, origin xyz=0.0 -0.1197 0.425 rpy=0.0 0.0 0.0, axis 0 -1.0 0, limit lower=-3.14159265359 upper=3.14159265359 effort=150.0 velocity=3.15
- added joint joint23: type revolute, parent link22, child link23, origin xyz=0.0 0.0 0.39225 rpy=0.0 1.57079632679 0.0, axis 0 1 0, limit lower=-6.28318530718 upper=6.28318530718 effort=28.0 velocity=3.2
- added joint joint24: type revolute, parent link23, child link24, origin xyz=0.0 0.093 0.0 rpy=0.0 0.0 0.0, axis 0 0 1, limit lower=-6.28318530718 upper=6.28318530718 effort=28.0 velocity=3.2
- added joint joint25: type revolute, parent link24, child link25, origin xyz=0.0 0.0 0.09465 rpy=0.0 0.0 0.0, axis 0 1 0, limit lower=-6.28318530718 upper=6.28318530718 effort=28.0 velocity=3.2
- added joint joint26: type revolute, parent link25, child link26, origin xyz=0.0 0.0 0.089159 rpy=0.0 0.0 0.0, axis 0 0 1, limit lower=-6.28318530718 upper=6.28318530718 effort=150.0 velocity=3.15
- added joint joint27: type revolute, parent link26, child link27, origin xyz=0.0 0.13585 0.0 rpy=0.0 1.57079632679 0.0, axis 1 0 0, limit lower=-6.28318530718 upper=6.28318530718 effort=150.0 velocity=3.15
- added joint joint28: type revolute, parent link27, child link28, origin xyz=0.0 -0.1197 0.425 rpy=0.0 0.0 0.0, axis 0 -1.0 0, limit lower=-3.14159265359 upper=3.14159265359 effort=150.0 velocity=3.15
- added joint joint29: type revolute, parent link28, child link29, origin xyz=0.0 0.0 0.39225 rpy=0.0 1.57079632679 0.0, axis 0 1 0, limit lower=-6.28318530718 upper=6.28318530718 effort=28.0 velocity=3.2
- added joint joint3: type revolute, parent link2, child link3, origin xyz=0.0 -0.1197 0.425 rpy=0.0 0.0 0.0, axis 0 1 0, limit lower=-3.14159265359 upper=3.14159265359 effort=150.0 velocity=3.15
- added joint joint30: type revolute, parent link29, child link30, origin xyz=0.0 0.093 0.0 rpy=0.0 0.0 0.0, axis 0 0 1, limit lower=-6.28318530718 upper=6.28318530718 effort=28.0 velocity=3.2
- added joint joint31: type revolute, parent link30, child link31, origin xyz=0.0 0.0 0.09465 rpy=0.0 0.0 0.0, axis 0 1 0, limit lower=-6.28318530718 upper=6.28318530718 effort=28.0 velocity=3.2
- added joint joint32: type revolute, parent link31, child link32, origin xyz=0.0 0.0 0.089159 rpy=0.0 0.0 0.0, axis 0 0 1, limit lower=-6.28318530718 upper=6.28318530718 effort=150.0 velocity=3.15
- added joint joint33: type revolute, parent link32, child link33, origin xyz=0.0 0.0 0.089159 rpy=0.0 0.0 0.0, axis 1 0 0, limit lower=-6.28318530718 upper=6.28318530718 effort=150.0 velocity=3.15
- added joint joint34: type revolute, parent link33, child link34, origin xyz=0.0 0.13585 0.0 rpy=0.0 1.57079632679 0.0, axis 1 0 0, limit lower=-6.28318530718 upper=6.28318530718 effort=150.0 velocity=3.15
- added joint joint4: type revolute, parent link3, child link4, origin xyz=0.0 0.0 0.39225 rpy=0.0 1.57079632679 0.0, axis 1 0 0, limit lower=-6.28318530718 upper=6.28318530718 effort=28.0 velocity=3.2
- added joint joint5: type revolute, parent link4, child link5, origin xyz=0.0 0.093 0.0 rpy=0.0 0.0 0.0, axis 1 0 0, limit lower=-6.28318530718 upper=6.28318530718 effort=28.0 velocity=3.2
- added joint joint6: type revolute, parent link5, child link6, origin xyz=0.0 0.0 0.09465 rpy=0.0 0.0 0.0, axis 1 0 0, limit lower=-6.28318530718 upper=6.28318530718 effort=28.0 velocity=3.2
- added joint joint7: type revolute, parent link6, child link7, origin xyz=0.0 0.13585 0.0 rpy=0.0 1.57079632679 0.0, axis 1 0 0, limit lower=-6.28318530718 upper=6.28318530718 effort=150.0 velocity=3.15
- added joint joint8: type revolute, parent link7, child link8, origin xyz=0.0 -0.1197 0.425 rpy=0.0 0.0 0.0, axis 0 1 0, limit lower=-3.14159265359 upper=3.14159265359 effort=150.0 velocity=3.15
- added joint joint9: type revolute, parent link8, child link9, origin xyz=0.0 0.0 0.39225 rpy=0.0 1.57079632679 0.0, axis 0 1 0, limit lower=-6.28318530718 upper=6.28318530718 effort=28.0 velocity=3.2

File: examples/timing/urdf4timing/35dof.urdf (robot description, URDF)
Before this commit: robot ur5, 35 links, 32 joints
Links:
- removed link forearm_link
- removed link shoulder_link
- removed link shoulder_link3
- removed link upper_arm_link
- removed link upper_arm_link2
- removed link wrist_1_link
- removed link wrist_2_link
- added link link1, mass 3.7; collision cylinder length=0.03 radius=0.2; visual cylinder length=0.03 radius=0.2
- added link link12, mass 3.7; collision cylinder length=0.03 radius=0.2; visual cylinder length=0.03 radius=0.2
- added link link2, mass 8.393; collision cylinder length=0.03 radius=0.2; visual cylinder length=0.03 radius=0.2
- added link link3, mass 2.275; collision cylinder length=0.03 radius=0.2; visual cylinder length=0.03 radius=0.2
- added link link35, mass 2.275; collision cylinder length=0.03 radius=0.2; visual cylinder length=0.03 radius=0.2
- added link link4, mass 1.219; collision cylinder length=0.03 radius=0.2; visual cylinder length=0.03 radius=0.2
- added link link5, mass 1.219; collision cylinder length=0.03 radius=0.2; visual cylinder length=0.03 radius=0.2
- added link link7, mass 8.393; collision cylinder length=0.03 radius=0.2; visual cylinder length=0.03 radius=0.2
- link link20: mass 8.393 -> 4.393
- link link33: mass 8.393 -> 3.7
- link link34: mass 2.275 -> 8.393
Joints:
- removed joint elbow_joint
- removed joint elbow_joint2
- removed joint elbow_joint3
- removed joint elbow_joint4
- removed joint elbow_joint5
- removed joint elbow_joint6
- removed joint shoulder_lift_joint
- removed joint shoulder_lift_joint2
- removed joint shoulder_lift_joint3
- removed joint shoulder_lift_joint4
- removed joint shoulder_lift_joint5
- removed joint shoulder_lift_joint6
- removed joint shoulder_pan_joint
- removed joint shoulder_pan_joint3
- removed joint shoulder_pan_joint4
- removed joint shoulder_pan_joint5
- removed joint shoulder_pan_joint6
- removed joint wrist_1_joint
- removed joint wrist_1_joint2
- removed joint wrist_1_joint3
- removed joint wrist_1_joint4
- removed joint wrist_1_joint5
- removed joint wrist_2_joint
- removed joint wrist_2_joint2
- removed joint wrist_2_joint3
- removed joint wrist_2_joint4
- removed joint wrist_2_joint5
- removed joint wrist_3_joint
- removed joint wrist_3_joint2
- removed joint wrist_3_joint3
- removed joint wrist_3_joint4
- removed joint wrist_3_joint5
- added joint joint1: type revolute, parent base_link, child link1, origin xyz=0.0 0.0 0.089159 rpy=0.0 0.0 0.0, axis 1 0 0, limit lower=-6.28318530718 upper=6.28318530718 effort=150.0 velocity=3.15
- added joint joint10: type revolute, parent link9, child link10, origin xyz=0.0 0.093 0.0 rpy=0.0 0.0 0.0, axis 0 0 1, limit lower=-6.28318530718 upper=6.28318530718 effort=28.0 velocity=3.2
- added joint joint11: type revolute, parent link10, child link11, origin xyz=0.0 0.0 0.09465 rpy=0.0 0.0 0.0, axis 0 1 0, limit lower=-6.28318530718 upper=6.28318530718 effort=28.0 velocity=3.2
- added joint joint12: type revolute, parent link11, child link12, origin xyz=0.0 0.0 0.089159 rpy=0.0 0.0 0.0, axis 0 0 1, limit lower=-6.28318530718 upper=6.28318530718 effort=150.0 velocity=3.15
- added joint joint13: type revolute, parent link12, child link13, origin xyz=0.0 0.13585 0.0 rpy=0.0 1.57079632679 0.0, axis 1 0 0, limit lower=-6.28318530718 upper=6.28318530718 effort=150.0 velocity=3.15
- added joint joint14: type revolute, parent link13, child link14, origin xyz=0.0 -0.1197 0.425 rpy=0.0 0.0 0.0, axis 0 -1.0 0, limit lower=-3.14159265359 upper=3.14159265359 effort=150.0 velocity=3.15
- added joint joint15: type revolute, parent link14, child link15, origin xyz=0.0 0.0 0.39225 rpy=0.0 1.57079632679 0.0, axis 0 1 0, limit lower=-6.28318530718 upper=6.28318530718 effort=28.0 velocity=3.2
- added joint joint16: type revolute, parent link15, child link16, origin xyz=0.0 0.093 0.0 rpy=0.0 0.0 0.0, axis 0 0 1, limit lower=-6.28318530718 upper=6.28318530718 effort=28.0 velocity=3.2
- added joint joint17: type revolute, parent link16, child link17, origin xyz=0.0 0.093 0.0 rpy=0.0 0.0 0.0, axis 0 0 1, limit lower=-6.28318530718 upper=6.28318530718 effort=28.0 velocity=3.2
- added joint joint18: type revolute, parent link17, child link18, origin xyz=0.0 0.0 0.09465 rpy=0.0 0.0 0.0, axis 0 1 0, limit lower=-6.28318530718 upper=6.28318530718 effort=28.0 velocity=3.2
- added joint joint19: type revolute, parent link18, child link19, origin xyz=0.0 0.0 0.089159 rpy=0.0 0.0 0.0, axis 0 0 1, limit lower=-6.28318530718 upper=6.28318530718 effort=150.0 velocity=3.15
- added joint joint2: type revolute, parent link1, child link2, origin xyz=0.0 0.13585 0.0 rpy=0.0 1.57079632679 0.0, axis 1 0 0, limit lower=-6.28318530718 upper=6.28318530718 effort=150.0 velocity=3.15
- added joint joint20: type revolute, parent link19, child link20, origin xyz=0.0 0.13585 0.0 rpy=0.0 1.57079632679 0.0, axis 1 0 0, limit lower=-6.28318530718 upper=6.28318530718 effort=150.0 velocity=3.15
- added joint joint21: type revolute, parent link20, child link21, origin xyz=0.0 0.13585 0.0 rpy=0.0 1.57079632679 0.0, axis 1 0 0, limit lower=-6.28318530718 upper=6.28318530718 effort=150.0 velocity=3.15
- added joint joint22: type revolute, parent link21, child link22, origin xyz=0.0 -0.1197 0.425 rpy=0.0 0.0 0.0, axis 0 -1.0 0, limit lower=-3.14159265359 upper=3.14159265359 effort=150.0 velocity=3.15
- added joint joint23: type revolute, parent link22, child link23, origin xyz=0.0 0.0 0.39225 rpy=0.0 1.57079632679 0.0, axis 0 1 0, limit lower=-6.28318530718 upper=6.28318530718 effort=28.0 velocity=3.2
- added joint joint24: type revolute, parent link23, child link24, origin xyz=0.0 0.093 0.0 rpy=0.0 0.0 0.0, axis 0 0 1, limit lower=-6.28318530718 upper=6.28318530718 effort=28.0 velocity=3.2
- added joint joint25: type revolute, parent link24, child link25, origin xyz=0.0 0.0 0.09465 rpy=0.0 0.0 0.0, axis 0 1 0, limit lower=-6.28318530718 upper=6.28318530718 effort=28.0 velocity=3.2
- added joint joint26: type revolute, parent link25, child link26, origin xyz=0.0 0.0 0.089159 rpy=0.0 0.0 0.0, axis 0 0 1, limit lower=-6.28318530718 upper=6.28318530718 effort=150.0 velocity=3.15
- added joint joint27: type revolute, parent link26, child link27, origin xyz=0.0 0.13585 0.0 rpy=0.0 1.57079632679 0.0, axis 1 0 0, limit lower=-6.28318530718 upper=6.28318530718 effort=150.0 velocity=3.15
- added joint joint28: type revolute, parent link27, child link28, origin xyz=0.0 -0.1197 0.425 rpy=0.0 0.0 0.0, axis 0 -1.0 0, limit lower=-3.14159265359 upper=3.14159265359 effort=150.0 velocity=3.15
- added joint joint29: type revolute, parent link28, child link29, origin xyz=0.0 0.0 0.39225 rpy=0.0 1.57079632679 0.0, axis 0 1 0, limit lower=-6.28318530718 upper=6.28318530718 effort=28.0 velocity=3.2
- added joint joint3: type revolute, parent link2, child link3, origin xyz=0.0 -0.1197 0.425 rpy=0.0 0.0 0.0, axis 0 1 0, limit lower=-3.14159265359 upper=3.14159265359 effort=150.0 velocity=3.15
- added joint joint30: type revolute, parent link29, child link30, origin xyz=0.0 0.093 0.0 rpy=0.0 0.0 0.0, axis 0 0 1, limit lower=-6.28318530718 upper=6.28318530718 effort=28.0 velocity=3.2
- added joint joint31: type revolute, parent link30, child link31, origin xyz=0.0 0.0 0.09465 rpy=0.0 0.0 0.0, axis 0 1 0, limit lower=-6.28318530718 upper=6.28318530718 effort=28.0 velocity=3.2
- added joint joint32: type revolute, parent link31, child link32, origin xyz=0.0 0.0 0.089159 rpy=0.0 0.0 0.0, axis 0 0 1, limit lower=-6.28318530718 upper=6.28318530718 effort=150.0 velocity=3.15
- added joint joint33: type revolute, parent link32, child link33, origin xyz=0.0 0.0 0.089159 rpy=0.0 0.0 0.0, axis 1 0 0, limit lower=-6.28318530718 upper=6.28318530718 effort=150.0 velocity=3.15
- added joint joint34: type revolute, parent link33, child link34, origin xyz=0.0 0.13585 0.0 rpy=0.0 1.57079632679 0.0, axis 1 0 0, limit lower=-6.28318530718 upper=6.28318530718 effort=150.0 velocity=3.15
- added joint joint35: type revolute, parent link34, child link35, origin xyz=0.0 -0.1197 0.425 rpy=0.0 0.0 0.0, axis 0 1 0, limit lower=-3.14159265359 upper=3.14159265359 effort=150.0 velocity=3.15
- added joint joint4: type revolute, parent link3, child link4, origin xyz=0.0 0.0 0.39225 rpy=0.0 1.57079632679 0.0, axis 1 0 0, limit lower=-6.28318530718 upper=6.28318530718 effort=28.0 velocity=3.2
- added joint joint5: type revolute, parent link4, child link5, origin xyz=0.0 0.093 0.0 rpy=0.0 0.0 0.0, axis 1 0 0, limit lower=-6.28318530718 upper=6.28318530718 effort=28.0 velocity=3.2
- added joint joint6: type revolute, parent link5, child link6, origin xyz=0.0 0.0 0.09465 rpy=0.0 0.0 0.0, axis 1 0 0, limit lower=-6.28318530718 upper=6.28318530718 effort=28.0 velocity=3.2
- added joint joint7: type revolute, parent link6, child link7, origin xyz=0.0 0.13585 0.0 rpy=0.0 1.57079632679 0.0, axis 1 0 0, limit lower=-6.28318530718 upper=6.28318530718 effort=150.0 velocity=3.15
- added joint joint8: type revolute, parent link7, child link8, origin xyz=0.0 -0.1197 0.425 rpy=0.0 0.0 0.0, axis 0 1 0, limit lower=-3.14159265359 upper=3.14159265359 effort=150.0 velocity=3.15
- added joint joint9: type revolute, parent link8, child link9, origin xyz=0.0 0.0 0.39225 rpy=0.0 1.57079632679 0.0, axis 0 1 0, limit lower=-6.28318530718 upper=6.28318530718 effort=28.0 velocity=3.2
