Commit message: timing

File: examples/timing/urdf4timing/2dof.urdf (robot description, URDF)
Before this commit: robot ur5, 3 links, 2 joints
Links:
- link base_link: mass 4.0 -> None; geometry 
- link link2: mass 8.393 -> 1; geometry 
- link shoulder_link: mass 3.7 -> 1; geometry 

File: examples/urdf/kuka.urdf (robot description, URDF)
Before this commit: robot kuka_lwr, 8 links, 7 joints
Links:
- link calib_kuka_arm_base_link: geometry 
- link kuka_arm_1_link: geometry 
- link kuka_arm_2_link: geometry 
- link kuka_arm_3_link: geometry 
- link kuka_arm_4_link: geometry 
- link kuka_arm_5_link: geometry 
- link kuka_arm_6_link: geometry 
- link kuka_arm_7_link: geometry 

File: examples/urdf/kukalwr.urdf (robot description, URDF)
Before this commit: robot kuka_lwr, 8 links, 7 joints
Joints:
- joint kuka_arm_0_joint: origin xyz=0 0 0.11 rpy=0 0 0 -> xyz=0 0 0.0 rpy=0 0 0
- joint kuka_arm_1_joint: origin xyz=0 0 0.20 rpy=0 0 0 -> xyz=0 0 0.0 rpy=0 0 0
- joint kuka_arm_2_joint: origin xyz=0 0 0.20 rpy=0 0 0 -> xyz=0 0 0.0 rpy=0 0 0
- joint kuka_arm_3_joint: origin xyz=0 0 0.20 rpy=0 0 0 -> xyz=0 0 0.0 rpy=0 0 0
- joint kuka_arm_4_joint: origin xyz=0 0 0.20 rpy=0 0 0 -> xyz=0 0 0.0 rpy=0 0 0
- joint kuka_arm_5_joint: origin xyz=0 0 0.19 rpy=0 0 0 -> xyz=0 0 0.0 rpy=0 0 0
- joint kuka_arm_6_joint: origin xyz=0 0 0.078 rpy=0 0 0 -> xyz=0 0 0.0 rpy=0 0 0

File: examples/urdf/pantilt.urdf (robot description, URDF)
Before this commit: robot pan_tilt, 3 links, 2 joints
Links:
- link base_link: mass None -> 1
- link tilt_link: mass 1 -> 5
Joints:
- joint pan_joint: axis 0 1 0 -> 0 0 1; limit lower=-3.14 upper=3.14 effort=300 velocity=1.0 -> lower=-3.14 upper=3.14 effort=300 velocity=0.1; origin xyz=0.0 0.0 1.0 rpy=0.0 0.0 0.0 -> xyz=0 0 0.1
- joint tilt_joint: origin xyz=0 0 1 rpy=0.0 0.0 0.0 -> xyz=4 0 1 rpy=0.0 0.0 0.0

File: examples/urdf/ur5_modified.urdf (robot description, URDF)
Before this commit: robot ur5, 7 links, 6 joints
Links:
- link base_link: mass 3.7 -> 4.0
